File: electronics/printer-board/printer-board/printer-board.kicad_pcb (KiCad board)
At the start: 2 copper layers, 125 x 63 mm, 38 parts, among them J1 XM, J10 THE1, J11 FAN1, J12 ZM1, J13 HE2, J14 THE2, J15 FAN2, J16 TFT, J17 EXP2, J18 EM0, J19 E0-Stop, J2 NeoPixel, J20 X-Stop, J21 EM1, J22 E1-Stop, J23 Y-Stop, J24 Bed, J25 I2C, J26 EM2, J27 E2-Stop, J28 Z-Stop, J29 Bed, J3 THB, J30 Hotend, J32 5V_PSU, J33 Hotend, J35 Extension1, J36 Extension2, J4 EXP1, J5 YM, J6 THE0, J7 FAN0, J8 BLTouch, J9 HE1

Commit message: updated routing
Parts:
- moved J10 1.68 mm to (167.0, 93.8)
- moved J21 1.68 mm to (195.0, 93.8)
- moved J25 1.68 mm to (181.0, 93.8)
- moved J11 1.00 mm to (195.2, 85.0)
- moved J22 1.00 mm to (176.5, 75.0)
- moved J6 1.00 mm to (185.8, 75.0)
- moved J7 1.00 mm to (195.2, 75.0)
- moved J8 1.00 mm to (186.0, 85.0)
Connections:
- J35 pad 10: unconnected-(J35-Pin_10-Pad10) -> HE2
- J35 pad 11: unconnected-(J35-Pin_11-Pad11) -> BLT_TRIGGER
- J35 pad 12: unconnected-(J35-Pin_12-Pad12) -> BLT_PWM
- J35 pad 13: unconnected-(J35-Pin_13-Pad13) -> VCC
- J35 pad 14: unconnected-(J35-Pin_14-Pad14) -> FAN2
- J35 pad 15: unconnected-(J35-Pin_15-Pad15) -> SDA
- J35 pad 16: unconnected-(J35-Pin_16-Pad16) -> SCL
- J35 pad 17: unconnected-(J35-Pin_17-Pad17) -> E1-STOP
- J35 pad 19: unconnected-(J35-Pin_19-Pad19) -> +3V3
- J35 pad 2: unconnected-(J35-Pin_2-Pad2) -> VCC
- J35 pad 21: Z-STOP -> GND
- J35 pad 23: unconnected-(J35-Pin_23-Pad23) -> +5V
- J35 pad 24: unconnected-(J35-Pin_24-Pad24) -> +3V3
- J35 pad 25: unconnected-(J35-Pin_25-Pad25) -> THE1
- J35 pad 26: unconnected-(J35-Pin_26-Pad26) -> THE2
- J35 pad 4: unconnected-(J35-Pin_4-Pad4) -> HE1
- J35 pad 6: unconnected-(J35-Pin_6-Pad6) -> FAN1
- J35 pad 8: unconnected-(J35-Pin_8-Pad8) -> FAN0
- J35 pad 9: unconnected-(J35-Pin_9-Pad9) -> THE0
- J36 pad 16: unconnected-(J36-Pin_16-Pad16) -> Z-STOP
Routing:
- net +3V3: track 0.00 -> 247.1 mm
- net +5V: track 16.4 -> 124.1 mm
- net Z-STOP: track 0.00 -> 105.5 mm
- net VCC: track 0.00 -> 73.4 mm
- net FAN0: track 0.00 -> 58.7 mm
- net FAN1: track 0.00 -> 45.4 mm
- net E1-STOP: track 0.00 -> 44.7 mm
- net THE0: track 0.00 -> 43.2 mm
- net BLT_TRIGGER: track 0.00 -> 38.8 mm
- net BLT_PWM: track 0.00 -> 37.4 mm
- net SCL: track 0.00 -> 26.5 mm
- net THE1: track 0.00 -> 24.0 mm
- net SDA: track 0.00 -> 23.0 mm
- net HE1: track 0.00 -> 16.1 mm
- net THE2: track 0.00 -> 15.6 mm
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- added copper zone on B.Cu, net GND
- added copper zone on F.Cu, net GND
